Commit message: added physical values for the minibot

File: src/my_robot/urdf/my_robot.urdf (robot description, URDF)
Before this commit: robot my_robot, 5 links, 4 joints
Links:
- link base_link: mass None -> 0.600; geometry collision box size=0.6 0.4 0.2; visual box size=0.6 0.4 0.2
- link caster_wheel: mass None -> 0.025; geometry collision sphere radius=0.05; visual sphere radius=0.05
- link left_wheel: mass None -> 0.050; geometry collision cylinder length=0.05 radius=0.1; visual cylinder length=0.05 radius=0.1
- link right_wheel: mass None -> 0.050; geometry collision cylinder length=0.05 radius=0.1; visual cylinder length=0.05 radius=0.1

Commit message: Added differential drive logic to the bot

File: src/my_robot/urdf/my_robot.urdf (robot description, URDF)
Before this commit: robot my_robot, 5 links, 4 joints
Links:
- link base_footprint: mass None -> 0.001
